File: wakey-wakey.kicad_pcb (KiCad board)
At the start: 2 copper layers, 78 x 49 mm, 18 parts, among them J1 Display_Conn, J2 BAT_PWR, SW1 SW_Push, SW2 SW_Push, SW3 SW_Push, SW4 SW_Push, U1 XIAO-ESP32-C3-SMD

Commit message: Finished CAD
Parts:
- J1: footprint Connector_PinSocket_2.54mm:PinSocket_1x08_P2.54mm_Vertical -> Connector_PinHeader_2.54mm:PinHeader_1x08_P2.54mm_Vertical
- J2: footprint Connector_PinSocket_2.54mm:PinSocket_1x02_P2.54mm_Vertical -> Connector_PinHeader_2.54mm:PinHeader_1x03_P2.54mm_Vertical
- moved H3 9.00 mm to (129.0, 119.0)
- moved H4 9.00 mm to (181.0, 119.0)
Routing:
- net Net-(J2-Pin_2): track 6.11 -> 8.53 mm
- net /CP1: track 89.0 -> 91.1 mm
Other:
- board text added: "BAT"
- board text added: "DISPLAY"
