File: PCB/wakey-wakey.kicad_pcb (KiCad board)
At the start: 2 copper layers, 78 x 49 mm, 18 parts, among them J1 Display_Conn, J2 BAT_PWR, SW1 SW_Push, SW2 SW_Push, SW3 SW_Push, SW4 SW_Push, U1 XIAO-ESP32-C3-SMD

Commit message: Improvements to PCB and CAD export
Parts:
- J2: footprint Connector_PinHeader_2.54mm:PinHeader_1x03_P2.54mm_Vertical -> Connector_PinHeader_2.54mm:PinHeader_1x04_P2.54mm_Vertical
Connections:
- J2 pad 2: Net-(J2-Pin_2) -> GND
- J2 pad 3: Net-(J2-Pin_2) -> Net-(J2-Pin_3)
- R1 pad 2: Net-(J2-Pin_2) -> Net-(J2-Pin_3)
Routing:
- net Net-(J2-Pin_3): track 0.00 -> 9.24 mm
- net Net-(J2-Pin_2): track 8.53 -> 0.00 mm
- net GND: track 65.3 -> 68.3 mm
- net /CP1: track 91.1 -> 94.0 mm
Changed lines of the file:
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@@
 			(layers "*.Cu" "*.Mask")
 			(remove_unused_layers no)
-			(net "Net-(J2-Pin_2)")
+			(net "Net-(J2-Pin_3)")
 			(pintype "passive")
 		)
@@
 		(embedded_fonts no)
 	)
-	(footprint "Connector_PinHeader_2.54mm:PinHeader_1x03_P2.54mm_Vertical"
+	(footprint "Connector_PinHeader_2.54mm:PinHeader_1x04_P2.54mm_Vertical"
 		(layer "B.Cu")
 		(at 138.54 79 90)
-		(descr "Through hole straight pin header, 1x03, 2.54mm pitch, single row")
-		(tags "Through hole pin header THT 1x03 2.54mm single row")
+		(descr "Through hole straight pin header, 1x04, 2.54mm pitch, single row")
+		(tags "Through hole pin header THT 1x04 2.54mm single row")
 		(property "Reference" "J2"
 			(at 0 2.38 270)
@@
 		)
 		(property "Value" "BAT_PWR"
-			(at 0 -7.46 270)
+			(at 0 -10 270)
 			(layer "B.Fab")
 			(effects
@@
 			)
 		)
-		(property "Description" "Generic connector, single row, 01x03, script generated"
+		(property "Description" "Generic connector, single row, 01x04, script generated"
 			(at 0 0 270)
 			(layer "B.Fab")
@@
 			(unit
 				(name "A")
-				(pins "1" "2" "3")
+				(pins "1" "2" "3" "4")
 			)
 		)
@@
 		(duplicate_pad_numbers_are_jumpers no)
 		(fp_line
-			(start -1.38 -6.46)
-			(end 1.38 -6.46)
+			(start -1.38 -9)
+			(end 1.38 -9)
 			(stroke
 				(width 0.12)
@@
 		(fp_line
 			(start 1.38 -1.27)
-			(end 1.38 -6.46)
+			(end 1.38 -9)
 			(stroke
 				(width 0.12)
@@
 		(fp_line
 			(start -1.38 -1.27)
-			(end -1.38 -6.46)
+			(end -1.38 -9)
 			(stroke
 				(width 0.12)
@@
 		(fp_rect
 			(start -1.77 1.77)
-			(end 1.77 -6.85)
+			(end 1.77 -9.39)
 			(stroke
 				(width 0.05)
@@
 		)
 		(fp_line
-			(start 1.27 -6.35)
-			(end -1.27 -6.35)
+			(start 1.27 -8.89)
+			(end -1.27 -8.89)
 			(stroke
 				(width 0.1)
@@
 		)
 		(fp_line
-			(start -1.27 -6.35)
+			(start -1.27 -8.89)
 			(end -1.27 0.635)
 			(stroke
@@
 		(fp_line
 			(start 1.27 1.27)
-			(end 1.27 -6.35)
+			(end 1.27 -8.89)
 			(stroke
 				(width 0.1)
@@
 		)
 		(fp_text user "${REFERENCE}"
-			(at 0 -2.54 0)
+			(at 0 -3.81 0)
 			(layer "B.Fab")
 			(effects
@@
 			(layers "*.Cu" "*.Mask")
 			(remove_unused_layers no)
-			(net "Net-(J2-Pin_2)")
+			(net "GND")
 			(pinfunction "Pin_2_2")
 			(pintype "passive")
@@
 			(layers "*.Cu" "*.Mask")
 			(remove_unused_layers no)
-			(net "Net-(J2-Pin_2)")
+			(net "Net-(J2-Pin_3)")
 			(pinfunction "Pin_3_3")
 			(pintype "passive")
 		)
+		(pad "4" thru_hole circle
+			(at 0 -7.62 90)
+			(size 1.7 1.7)
+			(drill 1)
+			(layers "*.Cu" "*.Mask")
+			(remove_unused_layers no)
+			(net "Net-(J2-Pin_3)")
+			(pinfunction "Pin_4_4")
+			(pintype "passive")
+		)
 		(embedded_fonts no)
-		(model "${KICAD10_3DMODEL_DIR}/Connector_PinHeader_2.54mm.3dshapes/PinHeader_1x03_P2.54mm_Vertical.step"
+		(model "${KICAD10_3DMODEL_DIR}/Connector_PinHeader_2.54mm.3dshapes/PinHeader_1x04_P2.54mm_Vertical.step"
 			(offset
 				(xyz 0 0 0)
@@
 	)
 	(gr_text "BAT"
-		(at 136 82.5 0)
+		(at 135 82.5 0)
 		(layer "B.SilkS")
 		(effects
@@
 	)
 	(segment
-		(start 130.55 94.395634)
-		(end 130.55 79.268)
+		(start 129.5 93.345634)
+		(end 129.5 78)
 		(width 0.2)
 		(layer "F.Cu")
@@
 	)
 	(segment
-		(start 130.55 79.268)
-		(end 132 77.818)
+		(start 129.5 78)
+		(end 130.5 77)
 		(width 0.2)
 		(layer "F.Cu")
@@
 	)
 	(segment
-		(start 132 77.818)
-		(end 159.018 77.818)
+		(start 140.36 102.65)
+		(end 138.804366 102.65)
 		(width 0.2)
 		(layer "F.Cu")
@@
 	)
 	(segment
-		(start 140.36 102.65)
-		(end 138.804366 102.65)
+		(start 138.804366 102.65)
+		(end 129.5 93.345634)
 		(width 0.2)
 		(layer "F.Cu")
@@
 	)
 	(segment
-		(start 159.018 77.818)
+		(start 158.2 77)
 		(end 162.62 81.42)
 		(width 0.2)
@@
 	)
 	(segment
-		(start 138.804366 102.65)
-		(end 130.55 94.395634)
+		(start 130.5 77)
+		(end 158.2 77)
 		(width 0.2)
 		(layer "F.Cu")
@@
 	)
 	(segment
-		(start 135.45 80.05)
-		(end 135.45 84.88)
-		(width 0.2)
-		(layer "F.Cu")
-		(net "Net-(J2-Pin_2)")
-	)
-	(segment
-		(start 136 79)
-		(end 136 79.5)
-		(width 0.2)
-		(layer "F.Cu")
-		(net "Net-(J2-Pin_2)")
-	)
-	(segment
-		(start 136 79.5)
-		(end 135.45 80.05)
+		(start 135.45 84.88)
+		(end 135.45 80.99)
 		(width 0.2)
 		(layer "F.Cu")
-		(net "Net-(J2-Pin_2)")
+		(net "Net-(J2-Pin_3)")
 	)
 	(segment
-		(start 134.51 80.05)
-		(end 135.45 80.05)
+		(start 133.46 79)
+		(end 130.92 79)
 		(width 0.2)
 		(layer "F.Cu")
-		(net "Net-(J2-Pin_2)")
+		(net "Net-(J2-Pin_3)")
 	)
 	(segment
-		(start 133.46 79)
-		(end 134.51 80.05)
+		(start 135.45 80.99)
+		(end 133.46 79)
 		(width 0.2)
 		(layer "F.Cu")
-		(net "Net-(J2-Pin_2)")
+		(net "Net-(J2-Pin_3)")
 	)
 	(segment
@@
 	)
 	(segment
+		(start 138.54 79)
+		(end 138.54 83.92)
+		(width 0.2)
+		(layer "F.Cu")
+		(net "GND")
+	)
+	(segment
 		(start 143.92 84.88)
 		(end 147.38 81.42)
@@
 	)
 	(segment
-		(start 138.54 83.92)
-		(end 139.5 84.88)
+		(start 136 79)
+		(end 136 79.5)
 		(width 0.2)
 		(layer "F.Cu")
@@
 	)
 	(segment
-		(start 138.54 79)
-		(end 138.54 83.92)
+		(start 136 79)
+		(end 138.54 79)
+		(width 0.2)
+		(layer "F.Cu")
+		(net "GND")
+	)
+	(segment
+		(start 138.54 83.92)
+		(end 139.5 84.88)
 		(width 0.2)
 		(layer "F.Cu")
