File: PCB/wakey-wakey.kicad_sch (KiCad schematic)
At the start: 18 parts, among them J1 Display_Conn, J2 BAT_PWR, SW1 SW_Push, SW2 SW_Push, SW3 SW_Push, SW4 SW_Push, U1 XIAO-ESP32-C3-SMD

Commit message: Improvements to PCB and CAD export
Parts:
- J2: footprint Connector_PinHeader_2.54mm:PinHeader_1x03_P2.54mm_Vertical -> Connector_PinHeader_2.54mm:PinHeader_1x04_P2.54mm_Vertical; symbol Connector:Conn_01x03_Pin -> Connector:Conn_01x04_Pin
Connections:
- net GND: now also J2.2 (Pin_2)
- net at J2.3 (Pin_3), R1.2: now also J2.4 (Pin_4); no longer J2.2 (Pin_2)
Changed lines of the file:
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@@
 	)
 	(junction
-		(at 205.74 138.43)
+		(at 205.74 143.51)
 		(diameter 0)
 		(color 0 0 0 0)
@@
 		(color 0 0 0 0)
 	)
+	(junction
+		(at 205.74 135.89)
+		(diameter 0)
+		(color 0 0 0 0)
+	)
 	(no_connect
 		(at 137.16 73.66)
@@
 	(wire
 		(pts
-			(xy 205.74 133.35) (xy 205.74 138.43)
-		)
-		(stroke
-			(width 0)
-			(type default)
-		)
-	)
-	(wire
-		(pts
 			(xy 217.17 91.44) (xy 223.52 91.44)
 		)
@@
 	(wire
 		(pts
+			(xy 205.74 140.97) (xy 205.74 143.51)
+		)
+		(stroke
+			(width 0)
+			(type default)
+		)
+	)
+	(wire
+		(pts
+			(xy 205.74 135.89) (xy 205.74 138.43)
+		)
+		(stroke
+			(width 0)
+			(type default)
+		)
+	)
+	(wire
+		(pts
 			(xy 217.17 76.2) (xy 223.52 76.2)
 		)
@@
 	(wire
 		(pts
-			(xy 205.74 138.43) (xy 205.74 140.97)
-		)
-		(stroke
-			(width 0)
-			(type default)
-		)
-	)
-	(wire
-		(pts
 			(xy 55.88 83.82) (xy 62.23 83.82)
 		)
@@
 		(pts
 			(xy 217.17 86.36) (xy 223.52 86.36)
+		)
+		(stroke
+			(width 0)
+			(type default)
+		)
+	)
+	(wire
+		(pts
+			(xy 205.74 133.35) (xy 205.74 135.89)
 		)
 		(stroke
@@
 	)
 	(symbol
-		(lib_id "Connector:Conn_01x03_Pin")
+		(lib_id "Connector:Conn_01x04_Pin")
 		(at 210.82 140.97 180)
 		(unit 1)
@@
 		(fields_autoplaced yes)
 		(property "Reference" "J2"
-			(at 212.09 139.6999 0)
+			(at 212.09 138.4299 0)
 			(show_name no)
 			(do_not_autoplace no)
@@
 		)
 		(property "Value" "BAT_PWR"
-			(at 212.09 142.2399 0)
+			(at 212.09 140.9699 0)
 			(show_name no)
 			(do_not_autoplace no)
@@
 			)
 		)
-		(property "Footprint" "Connector_PinHeader_2.54mm:PinHeader_1x03_P2.54mm_Vertical"
+		(property "Footprint" "Connector_PinHeader_2.54mm:PinHeader_1x04_P2.54mm_Vertical"
 			(at 210.82 140.97 0)
 			(hide yes)
@@
 			)
 		)
-		(property "Description" "Generic connector, single row, 01x03, script generated"
+		(property "Description" "Generic connector, single row, 01x04, script generated"
 			(at 210.82 140.97 0)
 			(hide yes)
@@
 		(pin "3"
 		)
+		(pin "4"
+		)
 		(instances
